File: display.kicad_sch (KiCad schematic)
At the start: 0 parts

Commit message: add lcd backlight driver, hierarchical signals to display page
Parts:
- added C20: 4.7uF, Capacitor_SMD:C_0402_1005Metric, symbol Device:C_Small
- added U11: AW9364DNR, custom:DFN-8_L2.0-W2.0-P0.50-BL-EP-1, symbol custom:AW9364DNR
Connections:
- new net +3V3: C20.1, U11.3 (VIN)
- new net BACKLIGHT_EN: U11.2 (EN)
- new net GND: C20.2, U11.1 (PGND), U11.4 (AGND), U11.9 (EP)
- new net LEDK1: U11.8 (LED1)
- new net LEDK2: U11.7 (LED2)
- new net LEDK3: U11.6 (LED3)
- new net LEDK4: U11.5 (LED4)
