File: display.kicad_sch (KiCad schematic)
At the start: 0 parts

Commit message: Display (#4)
* add lcd backlight driver, hierarchical signals to display page

* update ioc with backlight signals

* Add FPC library

* Add logic level shifters
Parts:
- added C20: 4.7uF, Capacitor_SMD:C_0402_1005Metric, symbol Device:C_Small
- added J12: YTC05201-500R-0WLW, custom:FPC-SMD_50P-P0.50_YTC05201-500R-0WLW, symbol custom:YTC05201-500R-0WLW
- added U11: AW9364DNR, custom:DFN-8_L2.0-W2.0-P0.50-BL-EP-1, symbol custom:AW9364DNR
- added U12, U13, U14: FXLA108BQX, custom:DHVQFN-20_L4.5-W2.5-P0.50-BL-EP, symbol custom:FXLA108BQX
Connections:
- new net +1V8: J12.40, J12.41, J12.7, J12.8, U12.20 (VCCB), U13.20 (VCCB), U14.20 (VCCB)
- new net +3V3: C20.1, J12.1, J12.42, U11.3 (VIN), U12.1 (VCCA), U13.1 (VCCA), U14.1 (VCCA)
- new net BACKLIGHT_EN: U11.2 (EN)
- new net DB0: J12.32, U12.12 (B7)
- new net DB1: J12.31, U13.19 (B0)
- new net DB10: J12.22, U14.18 (B1)
- new net DB11: J12.21, U14.17 (B2)
- new net DB12: J12.20, U14.16 (B3)
- new net DB13: J12.19, U14.15 (B4)
- new net DB14: J12.18, U14.14 (B5)
- new net DB15: J12.17, U14.13 (B6)
- new net DB2: J12.30, U13.18 (B1)
- new net DB3: J12.29, U13.17 (B2)
- new net DB4: J12.28, U13.16 (B3)
- new net DB5: J12.27, U13.15 (B4)
- new net DB6: J12.26, U13.14 (B5)
- new net DB7: J12.25, U13.13 (B6)
- new net DB8: J12.24, U13.12 (B7)
- new net DB9: J12.23, U14.19 (B0)
- new net DC: J12.37, U12.15 (B4)
- new net GND: C20.2, J12.11, J12.12, J12.13, J12.14, J12.15, J12.16, J12.34, J12.43, J12.48, J12.49, J12.50, J12.6, J12.9, U11.1 (PGND), U11.4 (AGND), U11.9 (EP), U12.10 (GND), U12.11 (nOE), U13.10 (GND), U13.11 (nOE), U14.10 (GND), U14.11 (nOE)
- new net LCD.DB0: U12.9 (A7)
- new net LCD.DB1: U13.2 (A0)
- new net LCD.DB10: U14.3 (A1)
- new net LCD.DB11: U14.4 (A2)
- new net LCD.DB12: U14.5 (A3)
- new net LCD.DB13: U14.6 (A4)
- new net LCD.DB14: U14.7 (A5)
- new net LCD.DB15: U14.8 (A6)
- new net LCD.DB2: U13.3 (A1)
- new net LCD.DB3: U13.4 (A2)
- new net LCD.DB4: U13.5 (A3)
- new net LCD.DB5: U13.6 (A4)
- new net LCD.DB6: U13.7 (A5)
- new net LCD.DB7: U13.8 (A6)
- new net LCD.DB8: U13.9 (A7)
- new net LCD.DB9: U14.2 (A0)
- new net LCD.DC: U12.6 (A4)
- new net LCD.RD: U12.8 (A6)
- new net LCD.TE: U12.4 (A2)
- new net LCD.WR: U12.7 (A5)
- new net LCD.nCS: U12.5 (A3)
- new net LCD.nRST: U14.9 (A7)
- new net LEDK1: J12.2, U11.8 (LED1)
- new net LEDK2: J12.3, U11.7 (LED2)
- new net LEDK3: J12.4, U11.6 (LED3)
- new net LEDK4: J12.5, U11.5 (LED4)
- new net RD: J12.35, U12.13 (B6)
- new net TE: J12.39, U12.17 (B2)
- new net WR: J12.36, U12.14 (B5)
- new net nCS: J12.38, U12.16 (B3)
- new net nRST: J12.10, U14.12 (B7)
- no-connect marks 0 -> 11
Other:
- note added: "CSX"
- note added: "D/CX(SCL)"
- note added: "DB0"
- note added: "DB1"
- note added: "DB10"
- note added: "DB11"
- note added: "DB12"
- note added: "DB13"
- note added: "DB14"
- note added: "DB15"
- note added: "DB16"
- note added: "DB17"
- note added: "DB2"
- note added: "DB3"
- note added: "DB4"
- note added: "DB5"
- note added: "DB6"
- note added: "DB7"
- note added: "DB8"
- note added: "DB9"
- note added: "DE"
- note added: "DOTCLK"
- note added: "GND"
- note added: "HSYNC"
- note added: "IM0"
- note added: "IM1"
- note added: "IM2"
- note added: "IM3"
- note added: "LEDA"
- note added: "LEDK1"
- note added: "LEDK2"
- note added: "LEDK3"
- note added: "LEDK4"
- note added: "NC"
- note added: "RD"
- note added: "RESET"
- note added: "SDA"
- note added: "TE"
- note added: "VCI"
- note added: "VDDI"
- note added: "VSYNC"
- note added: "WRX(D/CX)"
- note added: "XL(X-)/INT"
- note added: "XR(X+)/SCL"
- note added: "YD(Y+)/SDA"
- note added: "YU(Y-)/RESET"
